Commit message: Update URDF and meshes to improve potential ikfast solutionning

File: staubli_tx250_support/urdf/tx250.urdf (robot description, URDF)
Before this commit: robot staubli_tx250, 10 links, 10 joints
Joints:
- removed joint joint_6-tool0
- joint flange-tool0: origin xyz=0 0 0 rpy=0 1.57079632679 0 -> xyz=0 0 0 rpy=0 0 0
- joint joint_2: axis 0 0 1 -> 0 1 0; origin xyz=0.15 0 0 rpy=-1.5708 0 0 -> xyz=0.15 0 0 rpy=0 0 0
- joint joint_3: axis 0 0 1 -> 0 1 0; origin xyz=0 -1.025 0 rpy=0 0 0 -> xyz=0 0 1.025 rpy=0 0 0
- joint joint_4: origin xyz=0 -1.1558 0 rpy=1.5708 0 0 -> xyz=0 0 1.1558 rpy=0 0 0
- joint joint_5: axis 0 0 1 -> -1 0 1; origin xyz=-0.063781 0 0.10248 rpy=0 -0.7854 0 -> xyz=-0.063781 0 0.10248 rpy=0 0 0
- joint joint_6: origin xyz=0.063502 0 0.098102 rpy=0 0.7854 0 -> xyz=-0.02446589 0 0.11427128 rpy=0 0 0
- joint joint_6-flange: origin xyz=0 0 0 rpy=0 -1.57079632679 0 -> xyz=0 0 0 rpy=0 0 0

File: staubli_tx250_support/urdf/tx250_macro.xacro (robot description, xacro)
@@ -6,10 +6,10 @@
     <link  name="${prefix}base_link">
     <inertial>
-      <origin  xyz="0.007551 -5.3594E-05 0.18051"  rpy="-1.5708 0 0" />
+      <origin  xyz="0 0 0"  rpy="0 0 0" />
       <mass   value="22.973" />
       <inertia ixx="0"   ixy="0"   ixz="0" iyy="0"   iyz="0"   izz="0" />
     </inertial>
     <visual>
-      <origin  xyz="0 0 0"  rpy="-1.5708 0 0" />
+      <origin  xyz="0 0 0"  rpy="0 0 0" />
       <geometry>
         <mesh
@@ -21,5 +21,5 @@
     </visual>
     <collision>
-      <origin  xyz="0 0 0"  rpy="-1.5708 0 0" />
+      <origin  xyz="0 0 0"  rpy="0 0 0" />
       <geometry>
         <mesh
@@ -30,5 +30,5 @@
   <link  name="${prefix}link_1">
     <inertial>
-      <origin  xyz="0.085478 -0.0025471 -0.040487"  rpy="0 0 0" />
+      <origin  xyz="0 0 0"  rpy="0 0 0" />
       <mass   value="45.357" />
       <inertia ixx="0"   ixy="0"   ixz="0" iyy="0"   iyz="0"   izz="0" />
@@ -54,5 +54,5 @@
   <link  name="${prefix}link_2">
     <inertial>
-      <origin  xyz="-4.2821E-06 -0.4373 0.26459"  rpy="0 0 0" />
+      <origin  xyz="0 0 0"  rpy="0 0 0" />
       <mass   value="60.896" />
       <inertia ixx="0"   ixy="0"   ixz="0" iyy="0"   iyz="0"   izz="0" />
@@ -78,5 +78,5 @@
   <link  name="${prefix}link_3">
     <inertial>
-      <origin  xyz="0.0053614 -0.18215 -0.0015935"  rpy="0 0 0" />
+      <origin  xyz="0 0 0"  rpy="0 0 0" />
       <mass   value="41.321" />
       <inertia ixx="0"   ixy="0"   ixz="0" iyy="0"   iyz="0"   izz="0" />
@@ -102,5 +102,5 @@
   <link  name="${prefix}link_4">
     <inertial>
-      <origin  xyz="-0.014458 -2.0763E-05 0.057777"  rpy="0 0 0" />
+      <origin  xyz="0 0 0"  rpy="0 0 0" />
       <mass   value="2.2667" />
       <inertia ixx="0"   ixy="0"   ixz="0" iyy="0"   iyz="0"   izz="0" />
@@ -126,5 +126,5 @@
   <link  name="${prefix}link_5">
     <inertial>
-      <origin  xyz="0.0094371 -3.6945E-07 0.048577"  rpy="0 0 0" />
+      <origin  xyz="0 0 0"  rpy="0 0 0" />
       <mass   value="1.3104" />
       <inertia ixx="0"   ixy="0"   ixz="0" iyy="0"   iyz="0"   izz="0" />
@@ -150,5 +150,5 @@
   <link  name="${prefix}link_6">
     <inertial>
-      <origin  xyz="-1.4874E-05 2.3311E-11 -0.0057413"  rpy="0 0 0" />
+      <origin  xyz="0 0 0"  rpy="0 0 0" />
       <mass   value="0.081549" />
       <inertia ixx="0"   ixy="0"   ixz="0" iyy="0"   iyz="0"   izz="0" />
@@ -184,8 +184,8 @@
   </joint>
   <joint name="${prefix}joint_2"  type="revolute">
-    <origin  xyz="0.15 0 0" rpy="-1.5708 0 0" />
+    <origin  xyz="0.15 0 0" rpy="0 0 0" />
     <parent  link="link_1" />
     <child  link="link_2" />
-    <axis  xyz="0 0 1" />
+    <axis  xyz="0 1 0" />
     <limit
       lower="${radians(-137.5)}"
@@ -195,8 +195,8 @@
   </joint>
   <joint name="${prefix}joint_3"  type="revolute">
-    <origin  xyz="0 -1.025 0" rpy="0 0 0" />
+    <origin  xyz="0 0 1.025" rpy="0 0 0" />
     <parent  link="link_2" />
     <child  link="link_3" />
-    <axis  xyz="0 0 1" />
+    <axis  xyz="0 1 0" />
     <limit
       lower="${radians(-150)}"
@@ -206,5 +206,5 @@
   </joint>
   <joint name="${prefix}joint_4"  type="revolute">
-    <origin  xyz="0 -1.1558 0" rpy="1.5708 0 0" />
+    <origin  xyz="0 0 1.1558" rpy="0 0 0" />
     <parent  link="link_3" />
     <child  link="link_4" />
@@ -217,8 +217,8 @@
   </joint>
   <joint name="${prefix}joint_5"  type="revolute">
-    <origin  xyz="-0.063781 0 0.10248" rpy="0 -0.7854 0" />
+    <origin  xyz="-0.063781 0 0.10248" rpy="0 0 0" />
     <parent  link="link_4" />
     <child  link="link_5" />
-    <axis  xyz="0 0 1" />
+    <axis  xyz="-1 0 1" />
     <limit
       lower="${radians(-540)}"
@@ -228,5 +228,5 @@
   </joint>
   <joint name="${prefix}joint_6"  type="revolute">
-    <origin  xyz="0.063502 0 0.098102" rpy="0 0.7854 0" />
+    <origin  xyz="-0.02446589 0 0.11427128" rpy="0 0 0" />
     <parent  link="link_5" />
     <child  link="link_6" />
@@ -245,13 +245,13 @@
       <child link="${prefix}base"/>
     </joint>
-    <joint name="${prefix}joint_6-tool0" type="fixed">
+    <!--joint name="${prefix}joint_6-tool0" type="fixed">
       <parent link="${prefix}link_6"/>
       <child link="${prefix}tool0"/>
       <origin xyz="0 0 0" rpy="0 0 0"/>
-    </joint>
+    </joint-->
         <!-- ROS-Industrial 'flange' frame: attachment point for EEF models -->
     <link name="${prefix}flange" />
     <joint name="${prefix}joint_6-flange" type="fixed">
-      <origin xyz="0 0 0" rpy="0 ${radians(-90.0)} 0" />
+      <origin xyz="0 0 0" rpy="0 0 0" />
       <parent link="${prefix}link_6" />
       <child link="${prefix}flange" />
@@ -260,8 +260,8 @@
     <link name="${prefix}tool0" />
     <joint name="${prefix}flange-tool0" type="fixed">
-      <origin xyz="0 0 0" rpy="0 ${radians(90.0)} 0" />
+      <origin xyz="0 0 0" rpy="0 0 0" />
       <parent link="${prefix}flange" />
       <child link="${prefix}tool0" />
-    </joint>
+    </joint >
   </xacro:macro>
 </robot>
